File: spotmicroservo.brd (EAGLE design)
At the start: 25.4 x 39.4 mm, 39 parts, among them J1 B4B-PH-SM4-TB(LF)(SN), J2 CON_HEADER_1X02-B2B-XH-A(LF)(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

Commit message: Fix power path
Routing:
- net 5V: track 17.2 -> 27.1 mm
- net VIN: track 4.50 -> 12.2 mm
- removed copper zone on layer 1, net 5V
- removed copper zone on layer 1, net GND
- removed copper zone on layer 16, net GND
- removed copper zone on layer 1, net VIN
Changed lines of the file:
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@@
 <via x="93.345" y="53.975" extent="1-16" drill="0.35"/>
 <via x="95.5675" y="52.07" extent="1-16" drill="0.35"/>
-<polygon width="0.1524" layer="1">
-<vertex x="81.28" y="82.55"/>
-<vertex x="111.76" y="82.55"/>
-<vertex x="111.76" y="38.1"/>
-<vertex x="81.28" y="38.1"/>
-</polygon>
-<polygon width="0.1524" layer="16">
-<vertex x="78.74" y="85.09"/>
-<vertex x="114.3" y="85.09"/>
-<vertex x="114.3" y="35.56"/>
-<vertex x="78.74" y="35.56"/>
-</polygon>
 <wire x1="106.68" y1="73.025" x2="106.68" y2="71.12" width="0" layer="19" extent="1-1"/>
 <wire x1="106.68" y1="68.58" x2="106.68" y2="71.12" width="0" layer="19" extent="1-1"/>
@@
 <contactref element="U2" pad="2"/>
 <contactref element="R10" pad="1"/>
-<wire x1="104.14" y1="68.58" x2="104.14" y2="66.04" width="2.54" layer="1"/>
-<wire x1="104.14" y1="66.04" x2="104.14" y2="63.5" width="2.54" layer="1"/>
-<wire x1="104.14" y1="63.5" x2="104.14" y2="60.96" width="2.54" layer="1"/>
-<wire x1="104.14" y1="60.96" x2="104.14" y2="58.42" width="2.54" layer="1"/>
-<wire x1="104.14" y1="58.42" x2="104.14" y2="55.88" width="2.54" layer="1"/>
-<polygon width="0.0762" layer="1">
-<vertex x="102.87" y="55.88"/>
-<vertex x="102.87" y="54.9275" curve="-90"/>
-<vertex x="102.235" y="54.2925"/>
-<vertex x="96.8375" y="54.2925" curve="90"/>
-<vertex x="96.2025" y="53.6575"/>
-<vertex x="96.2025" y="51.7525"/>
-<vertex x="104.775" y="51.7525" curve="90"/>
-<vertex x="105.41" y="52.3875"/>
-<vertex x="105.41" y="55.88"/>
-</polygon>
+<wire x1="104.14" y1="68.58" x2="104.14" y2="66.04" width="1.905" layer="1"/>
+<wire x1="104.14" y1="66.04" x2="104.14" y2="63.5" width="1.905" layer="1"/>
+<wire x1="104.14" y1="63.5" x2="104.14" y2="60.96" width="1.905" layer="1"/>
+<wire x1="104.14" y1="60.96" x2="104.14" y2="58.42" width="1.905" layer="1"/>
+<wire x1="104.14" y1="58.42" x2="104.14" y2="55.88" width="1.905" layer="1"/>
 <wire x1="94.645" y1="49.84" x2="94.6525" y2="49.8475" width="0.3048" layer="1"/>
 <wire x1="94.6525" y1="49.8475" x2="95.885" y2="49.8475" width="0.3048" layer="1"/>
 <wire x1="97.79" y1="52.33" x2="97.79" y2="51.7525" width="0.3048" layer="1"/>
 <wire x1="97.79" y1="51.7525" x2="95.885" y2="49.8475" width="0.3048" layer="1"/>
-<wire x1="97.79" y1="52.33" x2="104.14" y2="55.88" width="0" layer="19" extent="1-1"/>
+<wire x1="104.14" y1="55.88" x2="104.14" y2="53.34" width="1.905" layer="1"/>
+<wire x1="97.79" y1="53.34" x2="97.79" y2="52.33" width="0.6096" layer="1"/>
+<wire x1="104.14" y1="53.34" x2="97.79" y2="53.34" width="1.905" layer="1"/>
 </signal>
 <signal name="N$1">
@@
 <contactref element="U2" pad="1"/>
 <contactref element="R10" pad="2"/>
-<polygon width="0.0762" layer="1">
-<vertex x="101.6" y="50.4825" curve="-90"/>
-<vertex x="102.235" y="51.1175"/>
-<vertex x="103.505" y="51.1175" curve="-90"/>
-<vertex x="104.14" y="50.4825"/>
-<vertex x="104.14" y="48.26" curve="-90"/>
-<vertex x="101.6" y="45.72"/>
-<vertex x="96.2025" y="45.72"/>
-<vertex x="96.2025" y="47.625"/>
-<vertex x="99.3775" y="47.625" curve="90"/>
-<vertex x="101.6" y="49.8475"/>
-</polygon>
 <wire x1="94.645" y1="49.19" x2="95.9075" y2="49.19" width="0.3048" layer="1"/>
 <wire x1="97.79" y1="47.3075" x2="97.79" y2="46.73" width="0.3048" layer="1"/>
 <wire x1="95.9075" y1="49.19" x2="97.79" y2="47.3075" width="0.3048" layer="1"/>
-<wire x1="97.79" y1="46.73" x2="102.89" y2="50.275" width="0" layer="19" extent="1-1"/>
+<wire x1="102.89" y1="50.275" x2="102.89" y2="48.28" width="1.905" layer="1"/>
+<wire x1="101.34" y1="46.73" x2="97.79" y2="46.73" width="1.905" layer="1"/>
+<wire x1="102.89" y1="48.28" x2="101.34" y2="46.73" width="1.905" layer="1"/>
 </signal>
 <signal name="N$10">
